File: pcb/touch/touch.kicad_pcb (KiCad board)
At the start: 2 copper layers, 92.7 x 16.5 mm, 10 parts, among them J1 HEADER-1x05, U1 AT42QT1070

Commit message: Updated schematics
Parts:
- added LOGO-OSHW-150: OSHW, Symbols:LOGO-OSHW-150, B.Cu at (175.1, 107.8)
Routing:
- net Net-(R6-Pad1): track 13.5 -> 12.7 mm
Other:
- board text added: "CLKV2-PC-06"
- board text added: "REV. A"
