File: pcb/touch/touch.sch (KiCad schematic (older format))
At the start: 10 parts, among them J1 HEADER-1x05, U1 AT42QT1070

Commit message: Updated schematics
Connections:
- wire segments 40 -> 35
Other:
- moved on the sheet: C1, C2, J1, R1, R2, R3, R4, R5, R6, U1
